Commit message: feat: add JointState publisher and update robot description
- Added `JointStatePublisher_` to `KinematicsPublisher` to broadcast joint states on the `/joint_states` topic.
- Implemented `AngleCallback` logic to publish the `body_angle` joint position, enabling real-time visualization in RViz via `robot_state_publisher`.
- Updated the launch file to use `xacro` for processing the URDF, ensuring proper XML generation.
- Renamed and corrected joint axes in the XACRO file to align with the physical robot kinematics, specifically renaming the main articulation joint to `body_angle`.

File: src/robot_description/src/urdf/Floribot.urdf.xacro (robot description, xacro)
@@ -85,6 +85,6 @@
     </inertial>
   </link>
-  <joint name="body_angle" type="revolute">
-    <axis xyz="1 0 0"/>
+  <joint name="body_angle_pitch" type="revolute">
+    <axis xyz="0 1 0"/>
     <limit effort="1.0" lower="-1.57" upper="1.57" velocity="0.5"/>
     <parent link="axesFront"/>
@@ -113,5 +113,5 @@
     </inertial>
   </link>
-  <joint name="j_revolute_front_rear" type="revolute">
+  <joint name="body_angle" type="revolute">
     <axis xyz="0 0 1"/>
     <limit effort="1.0" lower="-1.57" upper="1.57" velocity="0.5"/>

Commit message: Update Floribot.urdf.xacro

File: src/robot_description/src/urdf/Floribot.urdf.xacro (robot description, xacro)
@@ -19,6 +19,6 @@
   <xacro:property name="wheel_joint_2_mid_joint" value="0.383" />
   <xacro:property name="sensor_z" value="0.36" />
-  <xacro:property name="front_sensor_x" value="-0.34" />
-  <xacro:property name="rear_sensor_x" value="0.34" />
+  <xacro:property name="front_sensor_x" value="0.34" />
+  <xacro:property name="rear_sensor_x" value="-0.34" />
   <xacro:property name="camera_z" value="0.47" />
   <!-- <xacro:property name="pi" value="3.141592653589793" /> Muss nicht definiert werden. -->

Commit message: changed link name lasers

File: src/robot_description/src/urdf/Floribot.urdf.xacro (robot description, xacro)
@@ -295,5 +295,5 @@
     </plugin>
   </gazebo>
-  <link name="front_laser_link">
+  <link name="sick_front_link">
     <visual>
       <origin xyz="0 0 0" rpy="0 0 0"/>
@@ -377,5 +377,5 @@
     <origin xyz="${rear_sensor_x} 0 ${sensor_z}" rpy="${pi} 0 ${pi}"/>
   </joint>
-  <gazebo reference="rear_laser_link">
+  <gazebo reference="sick_rear_link">
     <sensor name="rear_laser" type="gpu_lidar">
       <pose>0 0 0 0 0 0</pose>

Commit message: Revert "changed link name lasers"
This reverts commit b8823b28189da3e6e85316e1909ea7e76fae3be4.

File: src/robot_description/src/urdf/Floribot.urdf.xacro (robot description, xacro)
@@ -295,5 +295,5 @@
     </plugin>
   </gazebo>
-  <link name="sick_front_link">
+  <link name="front_laser_link">
     <visual>
       <origin xyz="0 0 0" rpy="0 0 0"/>
@@ -377,5 +377,5 @@
     <origin xyz="${rear_sensor_x} 0 ${sensor_z}" rpy="${pi} 0 ${pi}"/>
   </joint>
-  <gazebo reference="sick_rear_link">
+  <gazebo reference="rear_laser_link">
     <sensor name="rear_laser" type="gpu_lidar">
       <pose>0 0 0 0 0 0</pose>
